File: schematic/nes-keyboard.sch (KiCad schematic (older format))
At the start: 7 parts, among them SW1 SW-SPDT, U1 Rotary_Encoder, U4 Feather_RP2040, U5 128x32_I2C_OLED, U6 NeoKey_2x2, U7 NeoKey_2x2, U8 NeoKey_1x2_Col

Commit message: added electrical schematic and cad files
Connections:
- wire segments 69 -> 66
Changed lines of the file:
@@
 Wire Wire Line
 	1800 1350 1800 800
-Wire Wire Line
-	1800 800  3250 800
 Connection ~ 3300 800
 Wire Wire Line
@@
 	2700 2500 2600 2500
 Wire Wire Line
-	2600 2500 2600 900
-Wire Wire Line
-	2600 900  3400 900
-Connection ~ 3400 900
-Wire Wire Line
 	3000 1700 3000 1800
 Wire Wire Line
@@
 	3450 1700 3550 1700
 Wire Wire Line
-	3100 2600 3250 2600
+	1800 800  2600 800
 Wire Wire Line
-	3250 2600 3250 800
-Connection ~ 3250 800
+	2600 800  2600 2500
+Connection ~ 2600 800
 Wire Wire Line
-	3250 800  3300 800
+	2600 800  3300 800
 $EndSCHEMATC
